File: A1200KBv2.kicad_pcb (KiCad board)
At the start: 2 copper layers, 450 x 125 mm, 109 parts, among them J1 Conn_01x32_Female, J2 LED HDR, K1 ESC, K10 L.BLANK, K11 F1, K12 L.AMIGA, K13 2, K14 W, K15 A, K16 Z, K17 F2, K18 3, K19 E, K2 TILDE, K20 S, K21 X, K22 F3, K23 4, K24 R, K25 D, K26 C, K27 F4, K28 5, K29 T, K3 TAB, K30 F, K31 V, K32 SPACE SWITCH, K33 F5, K34 6, K35 Y, K36 G, K37 B, K38 7, K39 U, K4 CTRL, K40 H, K41 N, K42 F6, K43 8, K44 I, K45 J, K46 M, K47 9, K48 O, K49 K, K5 L.SHIFT, K50 LESSTHAN, K51 F7, K52 0, K53 P, K54 L, K55 GRTRTHAN, K56 F8, K57 MINUS, K58 L.CURLY, K59 COLON, K6 L.ALT, K60 QUESTION, K61 R.AMIGA, K62 F9, K63 PLUS, K64 R.CURLY, K65 ", K66 R.SHIFT, K67 R.ALT, K68 F10, K69 PIPE, K7 1, K70 R.BLANK, K71 RETURN, K72 BS, K73 LEFT, K74 DEL, K75 UP, K76 DOWN, K77 HELP, K78 RIGHT, K79 NUM_(, K8 Q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

Commit message: 10mm higher; keyboard connector out of the way
Parts:
- moved J1 24.7 mm to (192.8, 37.2)
Routing:
- net /4: track 635.2 -> 663.9 mm
- net /6: track 208.8 -> 235.5 mm
- net /5: track 384.6 -> 410.6 mm
- net /8: track 210.6 -> 236.3 mm
- net /2: track 448.6 -> 474.1 mm
- net /26: track 292.7 -> 318.0 mm, vias 2 -> 3
- net /3: track 507.8 -> 533.0 mm
- net /24: track 440.6 -> 465.5 mm, vias 3 -> 4
- net /16: track 634.6 -> 659.3 mm, vias 4 -> 5
- net /14: track 251.1 -> 275.8 mm, vias 1 -> 2
- net /20: track 467.1 -> 491.8 mm, vias 2 -> 3
- net /12: track 229.5 -> 254.2 mm, vias 1 -> 2
- net /18: track 543.2 -> 567.9 mm, vias 2 -> 3
- net /22: track 391.0 -> 415.7 mm
- net /15: track 566.6 -> 591.3 mm
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Other:
- board size 450 x 125 mm -> 450 x 135 mm
- board text added: "Mechanical keyboard for the A1200 - A1200KBv2 r6 for Gateron KS-33 low-profile switches, A1200.net case aeberbach 09/24 grayunicorn.com LICENSE: CC BY-NC-SA 4.0"
- board text removed: "Mechanical keyboard for the A1200 - A1200KBv2 r4 for Gateron KS-33 low-profile switches, A1200.net case aeberbach 07/24 grayunicorn.com LICENSE: CC BY-NC-SA 4.0"

Commit message: Revert "10mm higher; keyboard connector out of the way"
This reverts commit 7b7d121ea175ab04d54ee7bb06e71218aa1ce09d.
Parts:
- moved J1 24.7 mm to (192.8, 61.9)
Routing:
- net /4: track 663.9 -> 635.2 mm
- net /6: track 235.5 -> 208.8 mm
- net /5: track 410.6 -> 384.6 mm
- net /8: track 236.3 -> 210.6 mm
- net /2: track 474.1 -> 448.6 mm
- net /26: track 318.0 -> 292.7 mm, vias 3 -> 2
- net /3: track 533.0 -> 507.8 mm
- net /24: track 465.5 -> 440.6 mm, vias 4 -> 3
- net /16: track 659.3 -> 634.6 mm, vias 5 -> 4
- net /14: track 275.8 -> 251.1 mm, vias 2 -> 1
- net /20: track 491.8 -> 467.1 mm, vias 3 -> 2
- net /12: track 254.2 -> 229.5 mm, vias 2 -> 1
- net /18: track 567.9 -> 543.2 mm, vias 3 -> 2
- net /22: track 415.7 -> 391.0 mm
- net /15: track 591.3 -> 566.6 mm
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Other:
- board size 450 x 135 mm -> 450 x 125 mm
- board text added: "Mechanical keyboard for the A1200 - A1200KBv2 r4 for Gateron KS-33 low-profile switches, A1200.net case aeberbach 07/24 grayunicorn.com LICENSE: CC BY-NC-SA 4.0"
- board text removed: "Mechanical keyboard for the A1200 - A1200KBv2 r6 for Gateron KS-33 low-profile switches, A1200.net case aeberbach 09/24 grayunicorn.com LICENSE: CC BY-NC-SA 4.0"
